File: koplingskjema_pex1/noe.sch (KiCad schematic (older format))
At the start: 8 parts, among them U1 LF33_TO220

Commit message: Addded: LED to schematic
Parts:
- added D?: LED, symbol Device:LED
- added R?: R, symbol Device:R
Connections:
- net vcc: now also D?.1 (K)
- net at U?.26 (PC3): now also R?.2
- new net: D?.2 (A), R?.1
Changed lines of the file:
@@
 EESchema Schematic File Version 4
-EELAYER 30 0
+LIBS:noe-cache
+EELAYER 29 0
 EELAYER END
 $Descr A4 11693 8268
@@
 	1    0    0    -1
 $EndComp
+$Comp
+L Device:LED D?
+U 1 1 5D934177
+P 4250 3450
+F 0 "D?" V 4197 3528 50  0000 L CNN
+F 1 "LED" V 4288 3528 50  0000 L CNN
+F 2 "" H 4250 3450 50  0001 C CNN
+F 3 "~" H 4250 3450 50  0001 C CNN
+	1    4250 3450
+	0    1    1    0
+$EndComp
+$Comp
+L Device:R R?
+U 1 1 5D935AAC
+P 4250 3800
+F 0 "R?" H 4320 3846 50  0000 L CNN
+F 1 "R" H 4320 3755 50  0000 L CNN
+F 2 "" V 4180 3800 50  0001 C CNN
+F 3 "~" H 4250 3800 50  0001 C CNN
+	1    4250 3800
+	1    0    0    -1
+$EndComp
+Text GLabel 4250 3200 1    50   Input ~ 0
+vcc
+Wire Wire Line
+	4250 3300 4250 3200
+Wire Wire Line
+	4250 3600 4250 3650
+Wire Wire Line
+	3850 4050 4250 4050
+Wire Wire Line
+	4250 4050 4250 3950
 $EndSCHEMATC
