File: Exercise1/koplingskjema_pex1/noe.sch (KiCad schematic (older format))
At the start: 10 parts, among them U1 LF33_TO220

Commit message: Added: ATmega168_Datasheet
Parts:
- gave numbers to parts that had none: 7
Other:
- moved on the sheet: C1, C2, C3, C4, D1, D2, R1, R2, U1, U2
